Commit message: Reorganize

File: src/gym-foos/gym_foos/assets/FoosballTable2.urdf (robot description, URDF)
Before this commit: robot foosball_table, 36 links, 35 joints
Links:
- link rod1: geometry visual cylinder length=1.524000 radius=0.009525
- link rod1_man0: geometry collision box size=0.012700 0.025400 0.114300; visual box size=0.012700 0.025400 0.114300
- link rod1_man1: geometry collision box size=0.012700 0.025400 0.114300; visual box size=0.012700 0.025400 0.114300
- link rod1_man2: geometry collision box size=0.012700 0.025400 0.114300; visual box size=0.012700 0.025400 0.114300
- link rod2: geometry visual cylinder length=1.524000 radius=0.009525
- link rod2_man0: geometry collision box size=0.012700 0.025400 0.114300; visual box size=0.012700 0.025400 0.114300
- link rod2_man1: geometry collision box size=0.012700 0.025400 0.114300; visual box size=0.012700 0.025400 0.114300
- link rod3: geometry visual cylinder length=1.524000 radius=0.009525
- link rod3_man0: geometry collision box size=0.012700 0.025400 0.114300; visual box size=0.012700 0.025400 0.114300
- link rod3_man1: geometry collision box size=0.012700 0.025400 0.114300; visual box size=0.012700 0.025400 0.114300
- link rod3_man2: geometry collision box size=0.012700 0.025400 0.114300; visual box size=0.012700 0.025400 0.114300
- link rod4: geometry visual cylinder length=1.524000 radius=0.009525
- link rod4_man0: geometry collision box size=0.012700 0.025400 0.114300; visual box size=0.012700 0.025400 0.114300
- link rod4_man1: geometry collision box size=0.012700 0.025400 0.114300; visual box size=0.012700 0.025400 0.114300
- link rod4_man2: geometry collision box size=0.012700 0.025400 0.114300; visual box size=0.012700 0.025400 0.114300
- link rod4_man3: geometry collision box size=0.012700 0.025400 0.114300; visual box size=0.012700 0.025400 0.114300
- link rod4_man4: geometry collision box size=0.012700 0.025400 0.114300; visual box size=0.012700 0.025400 0.114300
- link rod5: geometry visual cylinder length=1.524000 radius=0.009525
- link rod5_man0: geometry collision box size=0.012700 0.025400 0.114300; visual box size=0.012700 0.025400 0.114300
- link rod5_man1: geometry collision box size=0.012700 0.025400 0.114300; visual box size=0.012700 0.025400 0.114300
- link rod5_man2: geometry collision box size=0.012700 0.025400 0.114300; visual box size=0.012700 0.025400 0.114300
- link rod5_man3: geometry collision box size=0.012700 0.025400 0.114300; visual box size=0.012700 0.025400 0.114300
- link rod5_man4: geometry collision box size=0.012700 0.025400 0.114300; visual box size=0.012700 0.025400 0.114300
- link rod6: geometry visual cylinder length=1.524000 radius=0.009525
- link rod6_man0: geometry collision box size=0.012700 0.025400 0.114300; visual box size=0.012700 0.025400 0.114300
- link rod6_man1: geometry collision box size=0.012700 0.025400 0.114300; visual box size=0.012700 0.025400 0.114300
- link rod6_man2: geometry collision box size=0.012700 0.025400 0.114300; visual box size=0.012700 0.025400 0.114300
- link rod7: geometry visual cylinder length=1.524000 radius=0.009525
- link rod7_man0: geometry collision box size=0.012700 0.025400 0.114300; visual box size=0.012700 0.025400 0.114300
- link rod7_man1: geometry collision box size=0.012700 0.025400 0.114300; visual box size=0.012700 0.025400 0.114300
- link rod8: geometry visual cylinder length=1.524000 radius=0.009525
- link rod8_man0: geometry collision box size=0.012700 0.025400 0.114300; visual box size=0.012700 0.025400 0.114300
- link rod8_man1: geometry collision box size=0.012700 0.025400 0.114300; visual box size=0.012700 0.025400 0.114300
- link rod8_man2: geometry collision box size=0.012700 0.025400 0.114300; visual box size=0.012700 0.025400 0.114300
- link table: geometry collision box size=0.025400 0.736600 0.107950; collision box size=0.025400 0.736600 0.107950
Joints:
- joint floor_joint: origin (none) -> xyz=0.000000 0.000000 0.000000 rpy=0 0 0
- joint rod1_man0_joint: origin (none) -> xyz=-0.533400 -0.206375 0.000000 rpy=0 0 0
- joint rod1_man1_joint: origin (none) -> xyz=0.000000 0.206375 0.000000 rpy=0 0 0
- joint rod1_man2_joint: origin (none) -> xyz=0.000000 0.412750 0.000000 rpy=0 0 0
- joint rod2_man0_joint: origin (none) -> xyz=-0.381000 -0.120650 0.000000 rpy=0 0 0
- joint rod2_man1_joint: origin (none) -> xyz=0.000000 0.241300 0.000000 rpy=0 0 0
- joint rod3_man0_joint: origin (none) -> xyz=-0.228600 -0.184150 0.000000 rpy=0 0 0
- joint rod3_man1_joint: origin (none) -> xyz=0.000000 0.184150 0.000000 rpy=0 0 0
- joint rod3_man2_joint: origin (none) -> xyz=0.000000 0.368300 0.000000 rpy=0 0 0
- joint rod4_man0_joint: origin (none) -> xyz=-0.076200 -0.241300 0.000000 rpy=0 0 0
- joint rod4_man1_joint: origin (none) -> xyz=0.000000 0.120650 0.000000 rpy=0 0 0
- joint rod4_man2_joint: origin (none) -> xyz=0.000000 0.241300 0.000000 rpy=0 0 0
- joint rod4_man3_joint: origin (none) -> xyz=0.000000 0.361950 0.000000 rpy=0 0 0
- joint rod4_man4_joint: origin (none) -> xyz=0.000000 0.482600 0.000000 rpy=0 0 0
- joint rod5_man0_joint: origin (none) -> xyz=0.076200 -0.241300 0.000000 rpy=0 0 0
- joint rod5_man1_joint: origin (none) -> xyz=0.000000 0.120650 0.000000 rpy=0 0 0
- joint rod5_man2_joint: origin (none) -> xyz=0.000000 0.241300 0.000000 rpy=0 0 0
- joint rod5_man3_joint: origin (none) -> xyz=0.000000 0.361950 0.000000 rpy=0 0 0
- joint rod5_man4_joint: origin (none) -> xyz=0.000000 0.482600 0.000000 rpy=0 0 0
- joint rod6_man0_joint: origin (none) -> xyz=0.228600 -0.184150 0.000000 rpy=0 0 0
- joint rod6_man1_joint: origin (none) -> xyz=0.000000 0.184150 0.000000 rpy=0 0 0
- joint rod6_man2_joint: origin (none) -> xyz=0.000000 0.368300 0.000000 rpy=0 0 0
- joint rod7_man0_joint: origin (none) -> xyz=0.381000 -0.120650 0.000000 rpy=0 0 0
- joint rod7_man1_joint: origin (none) -> xyz=0.000000 0.241300 0.000000 rpy=0 0 0
- joint rod8_man0_joint: origin (none) -> xyz=0.533400 -0.206375 0.000000 rpy=0 0 0
- joint rod8_man1_joint: origin (none) -> xyz=0.000000 0.206375 0.000000 rpy=0 0 0
- joint rod8_man2_joint: origin (none) -> xyz=0.000000 0.412750 0.000000 rpy=0 0 0
