Commit message: Add training logging, inertia

File: src/gym-foos/gym_foos/assets/FoosballBall.urdf (robot description, URDF)
Before this commit: robot foosball_table, 1 links, 0 joints
Links:
- link ball: mass None -> 1

File: src/gym-foos/gym_foos/assets/FoosballTable2.urdf (robot description, URDF)
Before this commit: robot foosball_table, 36 links, 35 joints
Links:
- link floor: mass None -> 1
- link rod1: mass None -> 1
- link rod1_man0: mass None -> 1; geometry collision box size=0.012700 0.025400 0.101600; visual box size=0.012700 0.025400 0.101600
- link rod1_man1: mass None -> 1; geometry collision box size=0.012700 0.025400 0.101600; visual box size=0.012700 0.025400 0.101600
- link rod1_man2: mass None -> 1; geometry collision box size=0.012700 0.025400 0.101600; visual box size=0.012700 0.025400 0.101600
- link rod2: mass None -> 1
- link rod2_man0: mass None -> 1; geometry collision box size=0.012700 0.025400 0.101600; visual box size=0.012700 0.025400 0.101600
- link rod2_man1: mass None -> 1; geometry collision box size=0.012700 0.025400 0.101600; visual box size=0.012700 0.025400 0.101600
- link rod3: mass None -> 1
- link rod3_man0: mass None -> 1; geometry collision box size=0.012700 0.025400 0.101600; visual box size=0.012700 0.025400 0.101600
- link rod3_man1: mass None -> 1; geometry collision box size=0.012700 0.025400 0.101600; visual box size=0.012700 0.025400 0.101600
- link rod3_man2: mass None -> 1; geometry collision box size=0.012700 0.025400 0.101600; visual box size=0.012700 0.025400 0.101600
- link rod4: mass None -> 1
- link rod4_man0: mass None -> 1; geometry collision box size=0.012700 0.025400 0.101600; visual box size=0.012700 0.025400 0.101600
- link rod4_man1: mass None -> 1; geometry collision box size=0.012700 0.025400 0.101600; visual box size=0.012700 0.025400 0.101600
- link rod4_man2: mass None -> 1; geometry collision box size=0.012700 0.025400 0.101600; visual box size=0.012700 0.025400 0.101600
- link rod4_man3: mass None -> 1; geometry collision box size=0.012700 0.025400 0.101600; visual box size=0.012700 0.025400 0.101600
- link rod4_man4: mass None -> 1; geometry collision box size=0.012700 0.025400 0.101600; visual box size=0.012700 0.025400 0.101600
- link rod5: mass None -> 1
- link rod5_man0: mass None -> 1; geometry collision box size=0.012700 0.025400 0.101600; visual box size=0.012700 0.025400 0.101600
- link rod5_man1: mass None -> 1; geometry collision box size=0.012700 0.025400 0.101600; visual box size=0.012700 0.025400 0.101600
- link rod5_man2: mass None -> 1; geometry collision box size=0.012700 0.025400 0.101600; visual box size=0.012700 0.025400 0.101600
- link rod5_man3: mass None -> 1; geometry collision box size=0.012700 0.025400 0.101600; visual box size=0.012700 0.025400 0.101600
- link rod5_man4: mass None -> 1; geometry collision box size=0.012700 0.025400 0.101600; visual box size=0.012700 0.025400 0.101600
- link rod6: mass None -> 1
- link rod6_man0: mass None -> 1; geometry collision box size=0.012700 0.025400 0.101600; visual box size=0.012700 0.025400 0.101600
- link rod6_man1: mass None -> 1; geometry collision box size=0.012700 0.025400 0.101600; visual box size=0.012700 0.025400 0.101600
- link rod6_man2: mass None -> 1; geometry collision box size=0.012700 0.025400 0.101600; visual box size=0.012700 0.025400 0.101600
- link rod7: mass None -> 1
- link rod7_man0: mass None -> 1; geometry collision box size=0.012700 0.025400 0.101600; visual box size=0.012700 0.025400 0.101600
- link rod7_man1: mass None -> 1; geometry collision box size=0.012700 0.025400 0.101600; visual box size=0.012700 0.025400 0.101600
- link rod8: mass None -> 1
- link rod8_man0: mass None -> 1; geometry collision box size=0.012700 0.025400 0.101600; visual box size=0.012700 0.025400 0.101600
- link rod8_man1: mass None -> 1; geometry collision box size=0.012700 0.025400 0.101600; visual box size=0.012700 0.025400 0.101600
- link rod8_man2: mass None -> 1; geometry collision box size=0.012700 0.025400 0.101600; visual box size=0.012700 0.025400 0.101600
- link table: mass None -> 1; geometry collision box size=0.025400 0.736600 0.158750; collision box size=0.025400 0.736600 0.158750
