Commit message: Set joint limits on rod translation

File: src/gym-foos/gym_foos/assets/FoosballTable.urdf (robot description, URDF)
Before this commit: robot foosball_table, 36 links, 35 joints
Joints:
- joint rod1_joint: limit effort=100 velocity=100 -> lower=-0.12382499999999999 upper=0.12382499999999999 effort=100 velocity=100
- joint rod2_joint: limit effort=100 velocity=100 -> lower=-0.20955 upper=0.20955 effort=100 velocity=100
- joint rod3_joint: limit effort=100 velocity=100 -> lower=-0.14605 upper=0.14605 effort=100 velocity=100
- joint rod4_joint: limit effort=100 velocity=100 -> lower=-0.08889999999999998 upper=0.08889999999999998 effort=100 velocity=100
- joint rod5_joint: limit effort=100 velocity=100 -> lower=-0.08889999999999998 upper=0.08889999999999998 effort=100 velocity=100
- joint rod6_joint: limit effort=100 velocity=100 -> lower=-0.14605 upper=0.14605 effort=100 velocity=100
- joint rod7_joint: limit effort=100 velocity=100 -> lower=-0.20955 upper=0.20955 effort=100 velocity=100
- joint rod8_joint: limit effort=100 velocity=100 -> lower=-0.12382499999999999 upper=0.12382499999999999 effort=100 velocity=100
